File: NerdHex-Gamma.kicad_pcb (KiCad board)
At the start: 6 copper layers, 110 x 200 mm, 284 parts, among them J1 Connector 02x01, J8 Conn_01x06, M1 Fan_4pin, M2 Fan_4pin, U1 AP3211, U10 EMC2302-1, U11 TXU0102-DCU, U12 TMP1075, U13 TMP1075, U14 TXU0304PW, U15 25MHz, U16 BM1370_mode1, U17 BM1370_mode1, U18 BM1370_mode1, U19 BM1370_mode1, U2 TPS53647, U20 BM1370_mode1, U21 BM1370_mode1, U3 MCP1824T-0802E, U4 CSD95472Q5MC, U5 CSD95472Q5MC, U6 CSD95472Q5MC, U7 CSD95472Q5MC, U8 MCP1824T-1202E, U9 T-Display-S3

Commit message: test
Parts:
- removed the REF** at (109.5, 210.0)
- removed the REF** at (60.5, 130.0)
- removed the REF** at (57.0, 123.0)
- removed the REF** at (57.0, 217.0)
- removed the REF** at (113.0, 217.0)
- removed the REF** at (113.0, 123.0)
- removed the REF** at (109.5, 130.0)
- removed the REF** at (60.5, 210.0)
- added ?: , , F.Cu at (66.5, 97.3)
- added ?: , , F.Cu at (63.9, 96.0)
- added ?: , , F.Cu at (66.5, 104.7)
- added ?: , , F.Cu at (63.9, 97.3)
- added ?: , , F.Cu at (65.2, 74.7)
- added ?: , , F.Cu at (66.5, 76.0)
- added ?: , , F.Cu at (65.2, 93.6)
- added ?: , , F.Cu at (63.9, 84.7)
- added ?: , , F.Cu at (63.9, 106.0)
- added ?: , , F.Cu at (65.2, 83.6)
- added ?: , , F.Cu at (65.2, 96.0)
- added ?: , , F.Cu at (66.5, 77.3)
- added ?: , , F.Cu at (65.2, 104.7)
- added ?: , , F.Cu at (65.2, 106.0)
- added ?: , , F.Cu at (63.9, 86.0)
- added ?: , , F.Cu at (66.5, 84.7)
- added ?: , , F.Cu at (63.9, 107.3)
- added ?: , , F.Cu at (63.9, 77.3)
- added ?: , , F.Cu at (66.5, 107.3)
- added ?: , , F.Cu at (66.5, 86.0)
- added ?: , , F.Cu at (63.9, 94.7)
- added ?: , , F.Cu at (66.5, 87.3)
- added ?: , , F.Cu at (65.2, 97.3)
- added ?: , , F.Cu at (65.2, 87.3)
- added ?: , , F.Cu at (65.2, 94.7)
- added ?: , , F.Cu at (65.2, 108.4)
- added ?: , , F.Cu at (65.2, 76.0)
- added ?: , , F.Cu at (63.9, 87.3)
- added ?: , , F.Cu at (63.9, 104.7)
- added ?: , , F.Cu at (65.2, 73.6)
- added ?: , , F.Cu at (66.5, 106.0)
- added ?: , , F.Cu at (65.2, 86.0)
- added ?: , , F.Cu at (65.2, 98.4)
- added ?: , , F.Cu at (66.5, 74.7)
- added ?: , , F.Cu at (63.9, 74.7)
- added ?: , , F.Cu at (65.2, 77.3)
- added ?: , , F.Cu at (63.9, 76.0)
- added ?: , , F.Cu at (65.2, 103.6)
- added ?: , , F.Cu at (65.2, 78.4)
- added ?: , , F.Cu at (66.5, 94.7)
- added ?: , , F.Cu at (65.2, 107.3)
- added ?: , , F.Cu at (66.5, 96.0)
- added ?: , , F.Cu at (65.2, 88.4)
- added ?: , , F.Cu at (65.2, 84.7)
- added REF**: Hole Threaded M4, myfootprints:Hole Threaded M4, F.Cu at (45.0, 130.0)
- added REF**: Hole Threaded M4, myfootprints:Hole Threaded M4, F.Cu at (45.0, 210.0)
- added REF**: Hole Threaded M4, myfootprints:Hole Threaded M4, F.Cu at (110.0, 210.0)
- added REF**: Hole Threaded M4, myfootprints:Hole Threaded M4, F.Cu at (60.0, 130.0)
- added REF**: Hole Threaded M4, myfootprints:Hole Threaded M4, F.Cu at (60.0, 210.0)
- added REF**: Hole Threaded M4, myfootprints:Hole Threaded M4, F.Cu at (125.0, 130.0)
- added REF**: Hole Threaded M4, myfootprints:Hole Threaded M4, F.Cu at (110.0, 130.0)
- added REF**: Hole Threaded M4, myfootprints:Hole Threaded M4, F.Cu at (125.0, 210.0)
- C3, C4, C42, C45, C48, C49, C5, C52, C53, C55, C58, C77, C79, C81, C83, C86, C87, C89, C91, C92, JP3, R2, R25, R26, R3: moved to B.Cu
- moved R48 263.0 mm to (160.3, 72.0)
- moved C100 261.1 mm to (154.3, 74.3)
- moved U15 255.5 mm to (152.3, 67.1)
- moved J8 223.6 mm to (116.3, 96.2), turned to -90 degrees
- moved C99 221.1 mm to (116.3, 86.5), turned to -90 degrees
- moved C98 219.9 mm to (116.3, 91.5), turned to 90 degrees
- moved U14 215.9 mm to (112.3, 89.0), turned to -90 degrees
- moved R15 203.6 mm to (129.8, 87.9), turned to 90 degrees
- moved C42 197.9 mm to (98.4, 77.3)
- moved C45 197.6 mm to (98.4, 80.6)
- moved C48 197.4 mm to (98.4, 83.9)
- moved C49 197.1 mm to (98.4, 87.2)
- moved C52 196.9 mm to (98.4, 90.5)
- moved L2 196.7 mm to (83.5, 94.8)
- moved C53 196.7 mm to (98.4, 93.8)
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Connections:
- F1 pad 3: (no net) -> Net-(F1-Pad1)
- F1 pad 4: (no net) -> +12V
Routing:
- net +5V: track 0.00 -> 196.0 mm, vias 0 -> 8
- net +12V: track 0.00 -> 192.3 mm, vias 0 -> 57
- net /Power/VSENSE-: track 0.00 -> 90.2 mm, vias 0 -> 2
- net /Power/VSENSE+: track 0.00 -> 89.6 mm, vias 0 -> 2
- net /Power/TPS_TSEN: track 0.00 -> 81.1 mm, vias 0 -> 5
- net /Power/FCCM: track 0.00 -> 74.5 mm, vias 0 -> 5
- net /Power/LDO_EN: track 0.00 -> 73.7 mm, vias 0 -> 2
- net /Power/TPS_CSP4: track 0.00 -> 66.3 mm, vias 0 -> 3
- net /BM1370-Chain/RESET: track 0.00 -> 59.4 mm, vias 0 -> 2
- net /Power/TPS_PWM4: track 0.00 -> 59.1 mm, vias 0 -> 2
- net /T-Display-S3/SDA: track 0.00 -> 51.0 mm, vias 0 -> 1
- net /T-Display-S3/SCL: track 0.00 -> 48.9 mm, vias 0 -> 1
- net /Power/TPS_PWM3: track 0.00 -> 47.8 mm, vias 0 -> 2
- net /Power/TPS_CSP3: track 0.00 -> 43.5 mm, vias 0 -> 2
- net /Power/TPS_PWM2: track 0.00 -> 37.5 mm, vias 0 -> 2
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- added copper zone on F.Cu, net +12V
- added copper zone on In1.Cu, net +12V
- added copper zone on In1.Cu, net +3V3
- added copper zone on In4.Cu, net +VRef
- added copper zone on B.Cu, net GND
- added copper zone on F.Cu, net GND
- added copper zone on In1.Cu, net GND
- added copper zone on In3.Cu, net GND
- added copper zone on In4.Cu, net GND
- added copper zone on F.Cu, net Net-(F1-Pad1)
- added copper zone on In1.Cu, net Net-(F1-Pad1)
- added copper zone on F.Cu, net Net-(U4-VSW)
- added copper zone on In1.Cu, net Net-(U4-VSW)
- added copper zone on F.Cu, net Net-(U5-VSW)
- added copper zone on In1.Cu, net Net-(U5-VSW)
- added copper zone on F.Cu, net Net-(U6-VSW)
- added copper zone on In1.Cu, net Net-(U6-VSW)
- added copper zone on F.Cu, net Net-(U7-VSW)
- added copper zone on In1.Cu, net Net-(U7-VSW)
- added copper zone on B.Cu, net VDD
- added copper zone on F.Cu, net VDD
- added copper zone on In1.Cu, net VDD
- added copper zone on In2.Cu, net VDD

Commit message: tmp
Parts:
- C96, C97, U13: moved to B.Cu
- moved U12 163.5 mm to (85.0, 170.0)
- moved C96 155.4 mm to (83.7, 170.0), turned to 180 degrees
- moved U13 100.8 mm to (65.2, 113.5)
- moved C97 94.3 mm to (68.9, 113.2)
- moved C100 31.9 mm to (156.5, 106.1)
- moved R48 31.9 mm to (162.6, 103.8)
- moved U15 31.9 mm to (154.6, 98.9)
Routing:
- net /T-Display-S3/SCL: track 48.9 -> 210.0 mm, vias 1 -> 3
- net /T-Display-S3/SDA: track 51.0 -> 209.1 mm, vias 1 -> 4
- net +3V3: track 26.0 -> 161.1 mm, vias 11 -> 13
- net +5V: track 196.0 -> 253.3 mm
- net /Power/VR_RDY: track 5.50 -> 41.2 mm, vias 0 -> 2
- net /BM1370-Chain/BM1370-1/RO: track 0.00 -> 12.2 mm
- net /BM1370-Chain/BM1370-1/NRSTI: track 0.00 -> 12.2 mm
- net /BM1370-Chain/BM1370-1/CLKI: track 0.00 -> 12.2 mm
- net /BM1370-Chain/BM1370-1/CI: track 0.00 -> 12.2 mm
- net /BM1370-Chain/BM1370-1/BI: track 0.00 -> 12.2 mm
- net GND: track 31.0 -> 40.3 mm, vias 112 -> 123
- net Net-(U2-VIN): track 6.99 -> 7.53 mm

Commit message: asictest
Parts:
- added ?: , , F.Cu at (70.0, 170.0)
- added ?: , , F.Cu at (70.0, 150.0)
- added ?: , , F.Cu at (100.1, 190.0)
- added ?: , , F.Cu at (70.0, 190.0)
- added REF**: open pad, Nerd8:open pad, B.Cu at (100.1, 150.0)
- added REF**: open pad, Nerd8:open pad, B.Cu at (100.1, 170.0)
- moved U19 0.34 mm to (100.0, 190.0)
Routing:
- net /BM1370-Chain/BM1370-4/RI: track 0.00 -> 12.2 mm
- net /BM1370-Chain/BM1370-4/NRSTO: track 0.00 -> 12.2 mm
- net /BM1370-Chain/BM1370-4/CO: track 0.00 -> 12.2 mm
- net /BM1370-Chain/BM1370-4/CLKO: track 0.00 -> 12.2 mm
- net /BM1370-Chain/BM1370-4/BO: track 0.00 -> 12.2 mm
- net /BM1370-Chain/BM1370-1/RO: track 12.2 -> 0.00 mm
- net /BM1370-Chain/BM1370-1/NRSTI: track 12.2 -> 0.00 mm
- net /BM1370-Chain/BM1370-1/CLKI: track 12.2 -> 0.00 mm
- net /BM1370-Chain/BM1370-1/CI: track 12.2 -> 0.00 mm
- net /BM1370-Chain/BM1370-1/BI: track 12.2 -> 0.00 mm
- net GND: track 40.3 -> 31.5 mm, vias 123 -> 298
- net VDD: vias 50 -> 110
