File: NerdHex-Gamma.kicad_pcb (KiCad board)
At the start: 6 copper layers, 110 x 200 mm, 340 parts, among them J1 Connector 02x01, J8 Conn_01x06, M1 Fan_4pin, M2 Fan_4pin, U1 AP3211, U10 EMC2302-1, U11 TXU0102-DCU, U12 TMP1075, U13 TMP1075, U14 TXU0304PW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

Commit message: connected 12V Input
Connections:
- J1 pad 2: Net-(F1-Pad1) -> Net-(F1-Pin_1)
