File: Power.kicad_sch (KiCad schematic)
At the start: 139 parts, among them J2 Conn_01x01, J3 Conn_01x01, U1 AP3211, U2 TPS53647, U3 MCP1824T-0802E, U4 CSD95472Q5MC, U5 CSD95472Q5MC, U6 CSD95472Q5MC, U7 CSD95472Q5MC, U8 MCP1824T-1202E

Commit message: Sense1-2
Parts:
- added JP4, JP5: SolderJumper_3_Open, Jumper:SolderJumper-3_P1.3mm_Open_RoundedPad1.0x1.5mm, symbol Jumper:SolderJumper_3_Open
- added R32, R35: 0, Resistor_SMD:R_0805_2012Metric, symbol Device:R
Connections:
- net GND: now also R35.2
- net VDD: now also R32.2
- net VSENSE+: now also JP4.2 (C); no longer R25.1
- net VSENSE-: now also JP5.2 (C); no longer R26.1
- new net VSENSE(1)+: JP4.3 (B), R25.1
- new net VSENSE(1)-: JP5.3 (B), R26.1
- new net VSENSE(2)+: JP4.1 (A), R32.1
- new net VSENSE(2)-: JP5.1 (A), R35.1

Commit message: 22
Parts:
- HS1: now left out of the parts list
- JP4, JP5, TP1: now not fitted
- R1: value 33.2k -> 49.9k; OrderNr RMCF0805FT33K2CT-ND -> 311-49.9KCRCT-ND
Other:
- note added: "for IMAX=120A"
- note removed: "for IMAX=180A"
Changed lines of the file:
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@@
 		)
 	)
-	(text "for IMAX=180A"
+	(text "for IMAX=120A"
 		(exclude_from_sim no)
 		(at 39.116 123.444 90)
@@
 		(in_bom no)
 		(on_board yes)
-		(dnp no)
+		(dnp yes)
 		(fields_autoplaced yes)
 		(property "Reference" "JP5"
@@
 		(in_bom no)
 		(on_board yes)
-		(dnp no)
+		(dnp yes)
 		(property "Reference" "JP4"
 			(at 25.146 147.574 90)
@@
 		(unit 1)
 		(exclude_from_sim yes)
-		(in_bom yes)
+		(in_bom no)
 		(on_board yes)
 		(dnp yes)
@@
 			)
 		)
-		(property "Value" "33.2k"
+		(property "Value" "49.9k"
 			(at 46.228 122.174 90)
 			(effects
@@
 			)
 		)
-		(property "Description" "RES 33.2K OHM 1% 1/8W 0805"
+		(property "Description" "RES 49.9K OHM 1% 1/8W 0805"
 			(at 41.656 122.174 0)
 			(effects
@@
 			)
 		)
-		(property "OrderNr" "RMCF0805FT33K2CT-ND"
+		(property "OrderNr" "311-49.9KCRCT-ND"
 			(at 41.656 122.174 90)
 			(effects
@@
 		(in_bom no)
 		(on_board yes)
-		(dnp no)
+		(dnp yes)
 		(property "Reference" "TP1"
 			(at 76.1492 216.9668 0)

Commit message: Bucktest 90
Parts:
- removed C68, C70: 330µ/4V, Capacitor_SMD:C_1210_3225Metric, symbol Device:C
- removed JP1: Disable Phase 4, Jumper:SolderJumper-2_P1.3mm_Open_RoundedPad1.0x1.5mm, symbol Jumper:SolderJumper_2_Open
- removed JP4, JP5: SolderJumper_3_Open, Jumper:SolderJumper-3_P1.3mm_Open_RoundedPad1.0x1.5mm, symbol Jumper:SolderJumper_3_Open
- removed R32, R35: 0, Resistor_SMD:R_0805_2012Metric, symbol Device:R
Connections:
- net VSENSE(1)+ is gone; now on net VSENSE+: R25.1
- net VSENSE(1)- is gone; now on net VSENSE-: R26.1
