File: NerdHex-Gamma.kicad_sch (KiCad schematic)
At the start: 3 parts, among them J1 Connector 02x01

Commit message: 1
Parts:
- F1: footprint 3568:FUSE_3568 -> 8Axe:Fuseholder Blade_3568
- J1: footprint CONN2_1102030_OST -> Nerd8:CONN2
Changed lines of the file:
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@@
 			)
 		)
-		(property "Footprint" "CONN2_1102030_OST"
+		(property "Footprint" "Nerd8:CONN2"
 			(at 53.848 63.754 0)
 			(effects
@@
 			)
 		)
-		(property "Footprint" "3568:FUSE_3568"
+		(property "Footprint" "8Axe:Fuseholder Blade_3568"
 			(at 81.788 56.134 0)
 			(effects

Commit message: Sense1-2
Parts:
- added H1: Threaded Inserts, symbol Mechanical:MountingHole
- F1: Manufacturer SMBJ12A -> 3568; OrderNr SMBJ12ALFCT-ND -> 36-3568-ND
- J1: OrderNr (none) -> ED2953-ND
Changed lines of the file:
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@@
+			)
+		)
+		(property "OrderNr" "ED2953-ND"
+			(at 62.484 58.674 0)
+			(effects
+				(font
+					(size 1.27 1.27)
+				)
+				(hide yes)
 			)
 		)
@@
 			)
 		)
-		(property "Description" ""
+		(property "Description" "Fuseholder Mini Blade"
 			(at 81.788 56.134 0)
 			(effects
@@
 			)
 		)
-		(property "Manufacturer" "SMBJ12A"
+		(property "Manufacturer" "3568"
 			(at 81.788 56.134 0)
 			(effects
@@
 			)
 		)
-		(property "OrderNr" "SMBJ12ALFCT-ND"
+		(property "OrderNr" "  36-3568-ND"
 			(at 81.788 56.134 0)
 			(effects
@@
 					(unit 1)
 				)
+			)
+		)
+	)
+	(symbol
+		(lib_id "Mechanical:MountingHole")
+		(at 25.908 151.892 0)
+		(unit 1)
+		(exclude_from_sim yes)
+		(in_bom no)
+		(on_board no)
+		(dnp no)
+		(fields_autoplaced yes)
+		(property "Reference" "H1"
+			(at 29.21 150.6219 0)
+			(effects
+				(font
+					(size 1.27 1.27)
+				)
+				(justify left)
+			)
+		)
+		(property "Value" "Threaded Inserts"
+			(at 29.21 153.1619 0)
+			(effects
+				(font
+					(size 1.27 1.27)
+				)
+				(justify left)
+			)
+		)
+		(property "Footprint" ""
+			(at 25.908 151.892 0)
+			(effects
+				(font
+					(size 1.27 1.27)
+				)
+				(hide yes)
+			)
+		)
+		(property "Datasheet" "~"
+			(at 25.908 151.892 0)
+			(effects
+				(font
+					(size 1.27 1.27)
+				)
+				(hide yes)
+			)
+		)
+		(property "Description" "-"
+			(at 25.908 151.892 0)
+			(effects
+				(font
+					(size 1.27 1.27)
+				)
+				(hide yes)
+			)
+		)
+		(property "Distributor" "D"
+			(at 25.908 151.892 0)
+			(effects
+				(font
+					(size 1.27 1.27)
+				)
+				(hide yes)
+			)
+		)
+		(property "OrderNr" "36-24949CT-ND"
+			(at 25.908 151.892 0)
+			(effects
+				(font
+					(size 1.27 1.27)
+				)
+				(hide yes)
+			)
+		)
+		(instances
+			(project ""
+				(path "/3156566e-65fb-4f3c-a391-b6970212fc69"
+					(reference "H1")
+					(unit 1)
+				)

Commit message: 22
Parts:
- F1: OrderNr 36-3568-ND -> 36-3568-ND
- H1: now in the parts list
- J1: footprint Nerd8:CONN2 -> myfootprints:CONN2
Changed lines of the file:
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@@
 			)
 		)
-		(property "Footprint" "Nerd8:CONN2"
+		(property "Footprint" "myfootprints:CONN2"
 			(at 53.848 63.754 0)
 			(effects
@@
 			)
 		)
-		(property "OrderNr" "  36-3568-ND"
+		(property "OrderNr" "36-3568-ND"
 			(at 81.788 56.134 0)
 			(effects
@@
 		(unit 1)
 		(exclude_from_sim yes)
-		(in_bom no)
+		(in_bom yes)
 		(on_board no)
 		(dnp no)
@@
 			)
 		)
-		(property "Description" "-"
+		(property "Description" "Threaded Inserts"
 			(at 25.908 151.892 0)
 			(effects

Commit message: Testrouting
Parts:
- F1: symbol Fuseholder Blade 3568:3568 -> Connector_Generic:Conn_02x02_Counter_Clockwise; MANUFACTURER (none) -> Keystone; MAXIMUM_PACKAGE_HEIGHT (none) -> 7.37 mm; PARTREV (none) -> C; SNAPEDA_PN (none) -> 3568; STANDARD (none) -> Manufacturer Recommendations
Connections:
- net Power/+12V: now also F1.4 (Pin_4)
- net at F1.1 (Pin_1), J1.2: now also F1.3 (Pin_3)
Changed lines of the file:
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@@
 		(color 0 0 0 0)
 	)
+	(junction
+		(at 90.424 56.134)
+		(diameter 0)
+		(color 0 0 0 0)
+	)
+	(junction
+		(at 73.406 56.134)
+		(diameter 0)
+		(color 0 0 0 0)
+	)
 	(wire
 		(pts
@@
 	(wire
 		(pts
+			(xy 87.884 58.674) (xy 90.424 58.674)
+		)
+		(stroke
+			(width 0)
+			(type default)
+		)
+	)
+	(wire
+		(pts
 			(xy 146.05 111.76) (xy 141.224 111.76)
 		)
@@
 	(wire
 		(pts
-			(xy 89.408 56.134) (xy 97.028 56.134)
+			(xy 87.884 56.134) (xy 90.424 56.134)
 		)
 		(stroke
@@
 	(wire
 		(pts
+			(xy 90.424 56.134) (xy 97.028 56.134)
+		)
+		(stroke
+			(width 0)
+			(type default)
+		)
+	)
+	(wire
+		(pts
+			(xy 73.406 56.134) (xy 75.184 56.134)
+		)
+		(stroke
+			(width 0)
+			(type default)
+		)
+	)
+	(wire
+		(pts
 			(xy 97.028 56.134) (xy 113.792 56.134)
 		)
@@
 	(wire
 		(pts
+			(xy 90.424 58.674) (xy 90.424 56.134)
+		)
+		(stroke
+			(width 0)
+			(type default)
+		)
+	)
+	(wire
+		(pts
+			(xy 73.406 56.134) (xy 73.406 58.674)
+		)
+		(stroke
+			(width 0)
+			(type default)
+		)
+	)
+	(wire
+		(pts
 			(xy 138.176 57.912) (xy 175.514 57.912)
 		)
@@
 	(wire
 		(pts
+			(xy 75.184 58.674) (xy 73.406 58.674)
+		)
+		(stroke
+			(width 0)
+			(type default)
+		)
+	)
+	(wire
+		(pts
 			(xy 97.028 68.834) (xy 97.028 75.692)
 		)
@@
 	(wire
 		(pts
-			(xy 62.484 56.134) (xy 74.168 56.134)
+			(xy 62.484 56.134) (xy 73.406 56.134)
 		)
 		(stroke
@@
 	)
 	(symbol
-		(lib_id "Fuseholder Blade 3568:3568")
-		(at 81.788 56.134 0)
+		(lib_id "Connector_Generic:Conn_02x02_Counter_Clockwise")
+		(at 80.264 56.134 0)
 		(unit 1)
 		(exclude_from_sim no)
@@
 		(fields_autoplaced yes)
 		(property "Reference" "F1"
-			(at 81.788 49.53 0)
+			(at 81.534 49.53 0)
 			(effects
 				(font
@@
 		)
 		(property "Value" "3568"
-			(at 81.788 52.07 0)
+			(at 81.534 52.07 0)
 			(effects
 				(font
@@
 		)
 		(property "Footprint" "8Axe:Fuseholder Blade_3568"
-			(at 81.788 56.134 0)
+			(at 80.264 56.134 0)
+			(effects
+				(font
+					(size 1.27 1.27)
+				)
+				(hide yes)
+			)
+		)
+		(property "Datasheet" "~"
+			(at 80.264 56.134 0)
+			(effects
+				(font
+					(size 1.27 1.27)
+				)
+				(hide yes)
+			)
+		)
+		(property "Description" "Generic connector, double row, 02x02, counter clockwise pin numbering scheme (similar to DIP package numbering), script generated (kicad-library-utils/schlib/autogen/connector/)"
+			(at 80.264 56.134 0)
+			(effects
+				(font
+					(size 1.27 1.27)
+				)
+				(hide yes)
+			)
+		)
+		(property "Manufacturer" "3568"
+			(at 80.264 56.134 0)
 			(effects
 				(font
@@
 			)
 		)
-		(property "Datasheet" ""
-			(at 81.788 56.134 0)
-			(effects
-				(font
-					(size 1.27 1.27)
-				)
-				(hide yes)
-			)
-		)
-		(property "Description" "Fuseholder Mini Blade"
-			(at 81.788 56.134 0)
-			(effects
-				(font
-					(size 1.27 1.27)
-				)
-				(hide yes)
-			)
-		)
-		(property "Manufacturer" "3568"
-			(at 81.788 56.134 0)
+		(property "Distributor" "D"
+			(at 80.264 56.134 0)
+			(effects
+				(font
+					(size 1.27 1.27)
+				)
+				(hide yes)
+			)
+		)
+		(property "OrderNr" "36-3568-ND"
+			(at 80.264 56.134 0)
+			(effects
+				(font
+					(size 1.27 1.27)
+				)
+				(hide yes)
+			)
+		)
+		(property "PARTREV" "C"
+			(at 80.264 56.134 0)
 			(effects
 				(font
@@
 			)
 		)
-		(property "Distributor" "D"
-			(at 81.788 56.134 0)
-			(effects
-				(font
-					(size 1.27 1.27)
-				)
-				(hide yes)
-			)
-		)
-		(property "OrderNr" "36-3568-ND"
-			(at 81.788 56.134 0)
-			(effects
-				(font
-					(size 1.27 1.27)
-				)
+		(property "MANUFACTURER" "Keystone"
+			(at 80.264 56.134 0)
+			(effects
+				(font
+					(size 1.27 1.27)
+				)
+				(justify bottom)
+				(hide yes)
+			)
+		)
+		(property "SNAPEDA_PN" "3568"
+			(at 80.264 56.134 0)
+			(effects
+				(font
+					(size 1.27 1.27)
+				)
+				(justify bottom)
+				(hide yes)
+			)
+		)
+		(property "MAXIMUM_PACKAGE_HEIGHT" "7.37 mm"
+			(at 80.264 56.134 0)
+			(effects
+				(font
+					(size 1.27 1.27)
+				)
+				(justify bottom)
+				(hide yes)
+			)
+		)
+		(property "STANDARD" "Manufacturer Recommendations"
+			(at 80.264 56.134 0)
+			(effects
+				(font
+					(size 1.27 1.27)
+				)
+				(justify bottom)
 				(hide yes)
 			)
@@
 		(pin "2"
 		)
+		(pin "3"
+		)
+		(pin "4"
+		)
 		(instances
