File: BM1370.kicad_sch (KiCad schematic)
At the start: 19 parts, among them U16 BM1370_mode1

Commit message: 1
Parts:
- renumbered C109 to C133, C101 to C134, C111 to C135, C102 to C136, C103 to C137, C113 to C138, C104 to C139, C116 to C140, C114 to C141, C105 to C142, C115 to C143, C106 to C144, C107 to C145, C108 to C146, C110 to C147, C112 to C148, R30 to R36, R31 to R37, U16 to U18
Changed lines of the file:
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@@
 		(dnp no)
 		(fields_autoplaced yes)
-		(property "Reference" "#PWR0207"
+		(property "Reference" "#PWR0248"
 			(at 135.89 141.478 0)
 			(effects
@@
 		(on_board yes)
 		(dnp no)
-		(property "Reference" "C113"
+		(property "Reference" "C138"
 			(at 125.603 140.843 0)
 			(effects
@@
 		(on_board yes)
 		(dnp no)
-		(property "Reference" "#U05"
+		(property "Reference" "#U014"
 			(at 111.252 97.79 0)
 			(effects
@@
 		(dnp no)
 		(fields_autoplaced yes)
-		(property "Reference" "#PWR0195"
+		(property "Reference" "#PWR0252"
 			(at 156.21 120.65 0)
 			(effects
@@
 		(on_board yes)
 		(dnp no)
-		(property "Reference" "C112"
+		(property "Reference" "C148"
 			(at 199.263 119.761 0)
 			(effects
@@
 		(on_board yes)
 		(dnp no)
-		(property "Reference" "R30"
+		(property "Reference" "R36"
 			(at 99.06 101.6 90)
 			(effects
@@
 		(dnp no)
 		(fields_autoplaced yes)
-		(property "Reference" "#PWR0206"
+		(property "Reference" "#PWR0243"
 			(at 124.968 154.178 0)
 			(effects
@@
 		(on_board yes)
 		(dnp no)
-		(property "Reference" "C107"
+		(property "Reference" "C145"
 			(at 171.45 57.15 90)
 			(effects
@@
 		(on_board yes)
 		(dnp no)
-		(property "Reference" "C102"
+		(property "Reference" "C136"
 			(at 96.52 57.15 90)
 			(effects
@@
 		(dnp no)
 		(fields_autoplaced yes)
-		(property "Reference" "#PWR0200"
+		(property "Reference" "#PWR0256"
 			(at 185.928 133.35 0)
 			(effects
@@
 		(on_board yes)
 		(dnp no)
-		(property "Reference" "#U08"
+		(property "Reference" "#U016"
 			(at 189.738 115.57 0)
 			(effects
@@
 		(on_board yes)
 		(dnp no)
-		(property "Reference" "C116"
+		(property "Reference" "C140"
 			(at 134.112 168.656 90)
 			(effects
@@
 		(on_board yes)
 		(dnp no)
-		(property "Reference" "C108"
+		(property "Reference" "C146"
 			(at 182.88 57.15 90)
 			(effects
@@
 		(dnp no)
 		(fields_autoplaced yes)
-		(property "Reference" "#PWR0209"
+		(property "Reference" "#PWR0250"
 			(at 148.844 141.732 0)
 			(effects
@@
 		(dnp no)
 		(fields_autoplaced yes)
-		(property "Reference" "#PWR0190"
+		(property "Reference" "#PWR0239"
 			(at 102.87 120.65 0)
 			(effects
@@
 		(dnp no)
 		(fields_autoplaced yes)
-		(property "Reference" "#PWR0210"
+		(property "Reference" "#PWR0251"
 			(at 148.844 154.432 0)
 			(effects
@@
 		(on_board yes)
 		(dnp no)
-		(property "Reference" "C115"
+		(property "Reference" "C143"
 			(at 149.479 141.097 0)
 			(effects
@@
 		(on_board yes)
 		(dnp no)
-		(property "Reference" "#U06"
+		(property "Reference" "#U015"
 			(at 161.29 105.41 0)
 			(effects
@@
 		(on_board yes)
 		(dnp no)
-		(property "Reference" "C111"
+		(property "Reference" "C135"
 			(at 91.059 126.873 0)
 			(effects
@@
 		(on_board yes)
 		(dnp no)
-		(property "Reference" "C105"
+		(property "Reference" "C142"
 			(at 144.145 57.15 90)
 			(effects
@@
 		(on_board yes)
 		(dnp no)
-		(property "Reference" "#PWR0212"
+		(property "Reference" "#PWR0245"
 			(at 135.382 181.61 0)
 			(effects
@@
 		(on_board yes)
 		(dnp no)
-		(property "Reference" "#PWR0196"
+		(property "Reference" "#PWR0253"
 			(at 156.21 104.14 0)
 			(effects
@@
 		(on_board yes)
 		(dnp no)
-		(property "Reference" "R31"
+		(property "Reference" "R37"
 			(at 170.434 94.742 90)
 			(effects
@@
 		(dnp no)
 		(fields_autoplaced yes)
-		(property "Reference" "#PWR0205"
+		(property "Reference" "#PWR0242"
 			(at 124.968 141.478 0)
 			(effects
@@
 		(dnp no)
 		(fields_autoplaced yes)
-		(property "Reference" "#PWR0193"
+		(property "Reference" "#PWR0246"
 			(at 135.89 60.96 0)
 			(effects
@@
 		(dnp no)
 		(fields_autoplaced yes)
-		(property "Reference" "#PWR0194"
+		(property "Reference" "#PWR0247"
 			(at 135.89 120.65 0)
 			(effects
@@
 		(on_board yes)
 		(dnp no)
-		(property "Reference" "C101"
+		(property "Reference" "C134"
 			(at 85.09 57.15 90)
 			(effects
@@
 		(on_board yes)
 		(dnp no)
-		(property "Reference" "#PWR0197"
+		(property "Reference" "#PWR0254"
 			(at 172.72 97.79 0)
 			(effects
@@
 		(dnp no)
 		(fields_autoplaced yes)
-		(property "Reference" "#PWR0192"
+		(property "Reference" "#PWR0241"
 			(at 116.84 120.65 0)
 			(effects
@@
 		(on_board yes)
 		(dnp no)
-		(property "Reference" "C103"
+		(property "Reference" "C137"
 			(at 107.95 57.15 90)
 			(effects
@@
 		(dnp no)
 		(fields_autoplaced yes)
-		(property "Reference" "#PWR0208"
+		(property "Reference" "#PWR0249"
 			(at 135.89 154.178 0)
 			(effects
@@
 		(on_board yes)
 		(dnp no)
-		(property "Reference" "#PWR0203"
+		(property "Reference" "#PWR0257"
 			(at 198.628 120.396 0)
 			(effects
@@
 		(on_board yes)
 		(dnp no)
-		(property "Reference" "#U07"
+		(property "Reference" "#U013"
 			(at 81.026 122.936 0)
 			(effects
@@
 		(dnp no)
 		(fields_autoplaced yes)
-		(property "Reference" "#PWR0204"
+		(property "Reference" "#PWR0258"
 			(at 198.628 133.096 0)
 			(effects
@@
 		(dnp no)
 		(fields_autoplaced yes)
-		(property "Reference" "#PWR0202"
+		(property "Reference" "#PWR0238"
 			(at 90.424 140.208 0)
 			(effects
@@
 		(on_board yes)
 		(dnp no)
-		(property "Reference" "#PWR0191"
+		(property "Reference" "#PWR0240"
 			(at 116.332 104.14 0)
 			(effects
@@
 		(on_board yes)
 		(dnp no)
-		(property "Reference" "C106"
+		(property "Reference" "C144"
 			(at 158.75 57.15 90)
 			(effects
@@
 		(dnp no)
 		(fields_autoplaced yes)
-		(property "Reference" "#PWR0211"
+		(property "Reference" "#PWR0244"
 			(at 135.382 165.862 0)
 			(effects
@@
 		(on_board yes)
 		(dnp no)
-		(property "Reference" "C109"
+		(property "Reference" "C133"
 			(at 83.058 124.968 0)
 			(effects
@@
 		(on_board yes)
 		(dnp no)
-		(property "Reference" "C110"
+		(property "Reference" "C147"
 			(at 191.516 118.618 0)
 			(effects
@@
 		(dnp no)
 		(fields_autoplaced yes)
-		(property "Reference" "#PWR0199"
+		(property "Reference" "#PWR0236"
 			(at 77.216 140.716 0)
 			(effects
@@
 		(on_board yes)
 		(dnp no)
-		(property "Reference" "C114"
+		(property "Reference" "C141"
 			(at 136.525 140.843 0)
 			(effects
@@
 		(on_board yes)
 		(dnp no)
-		(property "Reference" "U16"
+		(property "Reference" "U18"
 			(at 120.65 64.77 0)
 			(effects
@@
 		(on_board yes)
 		(dnp no)
-		(property "Reference" "#PWR0201"
+		(property "Reference" "#PWR0237"
 			(at 90.424 127.508 0)
 			(effects
@@
 		(on_board yes)
 		(dnp no)
-		(property "Reference" "C104"
+		(property "Reference" "C139"
 			(at 120.65 57.15 90)
 			(effects

Commit message: DRC GND Vias
Parts:
- U18: footprint Nerd8:BM1370 -> Eigene:BM1370
Changed lines of the file:
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@@
 			)
 		)
-		(property "Footprint" "Nerd8:BM1370"
+		(property "Footprint" "Eigene:BM1370"
 			(at 152.4 119.38 0)
 			(effects
