File: T-Display-S3.kicad_sch (KiCad schematic)
At the start: 20 parts, among them J4 Conn_01x12-Socket, J5 Conn_01x12-Socket, J6 Conn_01x12-Header, J7 Conn_01x12-Header, M1 Fan_4pin, M2 Fan_4pin, U10 EMC2302-1, U11 TXU0102-DCU, U12 TMP1075, U13 TMP1075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

Commit message: 1
Parts:
- U12, U13: footprint myfootprints:TMP1075-DRL -> Qaxe:TMP1075-DRL
Changed lines of the file:
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@@
 			)
 		)
-		(property "Footprint" "myfootprints:TMP1075-DRL"
+		(property "Footprint" "Qaxe:TMP1075-DRL"
 			(at 176.022 52.07 0)
 			(effects
@@
 			)
 		)
-		(property "Footprint" "myfootprints:TMP1075-DRL"
+		(property "Footprint" "Qaxe:TMP1075-DRL"
 			(at 176.022 80.01 0)
 			(effects

Commit message: 12V Input + i2c pullups
Parts:
- added R32, R35: 2.7k, Resistor_SMD:R_0805_2012Metric, symbol Device:R
Connections:
- net +3V3: now also R32.1, R35.1
- net SCL: now also R32.2
- net SDA: now also R35.2
